File: esp32_breakout_tht2/esp32_breakout.kicad_pcb (KiCad board)
At the start: 2 copper layers, 54.9 x 64 mm, 11 parts, among them J10 UART1, J23 s2, J24 s1, J25 S1_VCC, J26 S1_GND, J27 S2_VCC, J28 S2_GND, J6 I2C1, J7 I2C2, J8 I2C3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

Commit message: generated all the boards, touched up
Routing:
- net GND: track 195.7 -> 197.8 mm
