File: esp32_breakout_tht2_shield/esp32_breakout_shield.kicad_pcb (KiCad board)
At the start: 2 copper layers, 54.9 x 64 mm, 7 parts, among them J1 BAT, J21 SPI1, J23 s2, J24 s1

Commit message: generated all the boards, touched up
Changed lines of the file:
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@@
 			)
 		)
-		(fp_text user "${REFERENCE}"
-			(at 0 2.5 270)
-			(unlocked yes)
-			(layer "F.Fab")
-			(effects
-				(font
-					(size 1 1)
-					(thickness 0.15)
-				)
-			)
-		)
 		(pad "1" thru_hole circle
 			(at -9.039538 9.452038 270)
@@
 			)
 		)
-		(fp_text user "${REFERENCE}"
-			(at 5.715 3.175 0)
-			(unlocked yes)
-			(layer "F.Fab")
-			(effects
-				(font
-					(size 1 1)
-					(thickness 0.15)
-				)
-			)
-		)
 		(pad "1" thru_hole circle
 			(at -5.08 -3.81)
@@
 		)
 		(property "Value" "OLED_128X64_1.3_I2C"
-			(at -3.145 17.865 90)
+			(at 6.35 8.89 90)
 			(layer "F.Fab")
 			(effects
@@
 			(at 0 -2.38 0)
 			(layer "F.SilkS")
+			(hide yes)
 			(effects
 				(font
@@
 		)
 		(property "Value" "SPI1"
-			(at 0 15.08 0)
+			(at -3.81 11.43 0)
 			(layer "F.Fab")
 			(effects
@@
 			(layer "F.Fab")
 		)
-		(fp_text user "${REFERENCE}"
-			(at 0 6.35 90)
-			(layer "F.Fab")
-			(effects
-				(font
-					(size 1 1)
-					(thickness 0.15)
-				)
-			)
-		)
 		(pad "1" thru_hole circle
 			(at 0 0)
@@
 		)
 	)
-	(gr_text "X"
-		(at 11.786 54.6 0)
-		(layer "F.Fab")
-		(effects
-			(font
-				(size 1 1)
-				(thickness 0.15)
-			)
-		)
-	)
 	(gr_text "32"
 		(at 7.62 26.67 0)
@@
 		)
 	)
-	(gr_text "RX"
-		(at 11.43 7.62 90)
-		(layer "F.Fab")
-		(effects
-			(font
-				(size 1 1)
-				(thickness 0.15)
-			)
-		)
-	)
 	(gr_text "S_VN/ADC1_3"
 		(at 19.431 19.05 0)
@@
 	)
 	(gr_text "G"
-		(at 38.481 26.67 0)
+		(at 30.48 26.67 0)
 		(layer "F.Fab")
 		(effects
@@
 	)
 	(gr_text "VSPI_SCK"
-		(at 36.449 31.623 0)
+		(at 33.02 31.75 0)
 		(layer "F.Fab")
 		(effects
@@
 		)
 	)
-	(gr_text "X"
-		(at 11.913 52.06 0)
-		(layer "F.Fab")
-		(effects
-			(font
-				(size 1 1)
-				(thickness 0.15)
-			)
-		)
-	)
 	(gr_text "33"
 		(at 7.62 29.21 0)
@@
 	)
 	(gr_text "VSPI_SS"
-		(at 36.322 34.163 0)
+		(at 29.21 34.29 0)
 		(layer "F.Fab")
 		(effects
@@
 		)
 	)
-	(gr_text "G"
-		(at 6.35 6.985 0)
-		(layer "F.Fab")
-		(effects
-			(font
-				(size 1 1)
-				(thickness 0.15)
-			)
-		)
-	)
 	(gr_text "USB END\n"
 		(at 26.67 62.23 0)
@@
 		)
 	)
-	(gr_text "G"
-		(at 2.769 61.204 0)
-		(layer "F.Fab")
-		(effects
-			(font
-				(size 1 1)
-				(thickness 0.15)
-			)
-		)
-	)
 	(gr_text "EN"
 		(at 15.113 14.097 0)
@@
 	)
 	(gr_text "I2C_SDA"
-		(at 36.449 24.003 0)
-		(layer "F.Fab")
-		(effects
-			(font
-				(size 1 1)
-				(thickness 0.15)
-			)
-		)
-	)
-	(gr_text "12"
-		(at 11.405 42.027 0)
+		(at 31.75 24.13 0)
 		(layer "F.Fab")
 		(effects
@@
 		)
 	)
-	(gr_text "TX"
-		(at 13.97 7.62 90)
-		(layer "F.Fab")
-		(effects
-			(font
-				(size 1 1)
-				(thickness 0.15)
-			)
-		)
-	)
 	(gr_text "VSPI_MISO"
-		(at 35.433 29.21 0)
-		(layer "F.Fab")
-		(effects
-			(font
-				(size 1 1)
-				(thickness 0.15)
-			)
-		)
-	)
-	(gr_text "G"
-		(at 12.04 44.567 0)
+		(at 31.75 29.21 0)
 		(layer "F.Fab")
 		(effects
@@
 	)
 	(gr_text "14"
-		(at 11.532 39.36 0)
-		(layer "F.Fab")
-		(effects
-			(font
-				(size 1 1)
-				(thickness 0.15)
-			)
-		)
-	)
-	(gr_text "14"
 		(at 7.62 39.37 0)
 		(layer "F.Fab")
@@
 		)
 	)
-	(gr_text "3V3"
-		(at 8.89 7.62 90)
-		(layer "F.Fab")
-		(effects
-			(font
-				(size 1 1)
-				(thickness 0.15)
-			)
-		)
-	)
 	(gr_text "X"
 		(at 8.255 49.53 0)
@@
 		)
 	)
-	(gr_text "X"
-		(at 11.913 49.52 0)
-		(layer "F.Fab")
-		(effects
-			(font
-				(size 1 1)
-				(thickness 0.15)
-			)
-		)
-	)
 	(gr_text "EN"
 		(at 7.62 13.97 0)
@@
 		(start 38.1 60.96)
 		(end 25.4 60.96)
-		(width 1.016)
+		(width 0.762)
 		(layer "B.Cu")
 		(net 2)
@@
 		(start 25.4 60.96)
 		(end 18.372866 53.932866)
-		(width 1.016)
+		(width 0.762)
 		(layer "B.Cu")
 		(net 2)
@@
 		(start 38.1 39.37)
 		(end 38.1 60.96)
-		(width 1.016)
+		(width 0.762)
 		(layer "B.Cu")
 		(net 2)
@@
 		(start 40.66 11.41)
 		(end 38.1 13.97)
-		(width 0.889)
+		(width 0.635)
 		(layer "B.Cu")
 		(net 3)
@@
 		(start 35.32316 21.59)
 		(end 40.42316 16.49)
-		(width 0.889)
+		(width 0.635)
 		(layer "B.Cu")
 		(net 8)
@@
 		(start 40.42316 16.49)
 		(end 41.86 16.49)
-		(width 0.889)
+		(width 0.635)
 		(layer "B.Cu")
 		(net 8)
@@
 		(start 41.86 19.03)
 		(end 40.42316 19.03)
-		(width 0.889)
+		(width 0.635)
 		(layer "B.Cu")
 		(net 9)
@@
 		(start 31.75 27.70316)
 		(end 31.75 42.46452)
-		(width 0.889)
+		(width 0.635)
 		(layer "B.Cu")
 		(net 9)
@@
 		(start 31.75 42.46452)
 		(end 33.058346 43.772866)
-		(width 0.889)
+		(width 0.635)
 		(layer "B.Cu")
 		(net 9)
@@
 		(start 40.42316 19.03)
 		(end 31.75 27.70316)
-		(width 0.889)
+		(width 0.635)
 		(layer "B.Cu")
 		(net 9)
@@
 		(start 38.1 36.83)
 		(end 40.66 34.27)
-		(width 0.889)
+		(width 0.635)
 		(layer "B.Cu")
 		(net 12)
@@
 		(start 40.64 13.97)
 		(end 38.1 16.51)
-		(width 0.889)
+		(width 0.635)
 		(layer "B.Cu")
 		(net 13)
@@
 		(start 38.1 16.51)
 		(end 34.29 16.51)
-		(width 0.889)
+		(width 0.635)
 		(layer "B.Cu")
 		(net 13)
