File: sdcard_shield/sdcard_shield.kicad_sch (KiCad schematic)
At the start: 5 parts, among them J1 esp_23-5, J2 sd_reader, J3 PWR

Commit message: fixed it
Connections:
- net MISO: now also J1.3 (Pin_3); no longer J1.8 (Pin_8)
- net MOSI: now also J1.8 (Pin_8); no longer J1.3 (Pin_3)
Changed lines of the file:
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@@
 	(global_label "MISO"
 		(shape input)
-		(at 120.65 49.53 0)
+		(at 120.65 62.23 0)
 		(effects
 			(font
@@
 		)
 		(property "Intersheetrefs" "${INTERSHEET_REFS}"
-			(at 120.65 49.53 0)
+			(at 120.65 62.23 0)
 			(effects
 				(font
@@
 	(global_label "MOSI"
 		(shape input)
-		(at 120.65 62.23 0)
+		(at 120.65 49.53 0)
 		(effects
 			(font
@@
 		)
 		(property "Intersheetrefs" "${INTERSHEET_REFS}"
-			(at 120.65 62.23 0)
+			(at 120.65 49.53 0)
 			(effects
 				(font
